Commit message: add offset to inspire

File: robots/hands/inspire_hand/inspire_hand_left.urdf (robot description, URDF)
Before this commit: robot inspire_hand_left, 19 links, 18 joints
Links:
- added link base1
Joints:
- added joint base1: type fixed, parent base1, child base, origin xyz=0 0 -0.045 rpy=0 0 0

File: robots/hands/inspire_hand/inspire_hand_right.urdf (robot description, URDF)
Before this commit: robot inspire_hand_right, 19 links, 18 joints
Links:
- added link base1
Joints:
- added joint base1: type fixed, parent base1, child base, origin xyz=0 0 -0.045 rpy=0 0 0
